Commit message: Renamed rtabmap to mapping

File: catkin_ws/src/my_robot/urdf/my_robot.xacro (robot description, xacro)
@@ -123,4 +123,5 @@
     <dynamics damping="1.0" friction="1.0"/>
   </joint>
+  <!-- Camera -->
   <link name="camera">
     <pose>0 0 0 0 0 0</pose>
@@ -155,4 +156,12 @@
     <dynamics damping="1.0" friction="1.0"/>
   </joint>
+  <joint name="camera_optical_joint" type="fixed">
+    <origin xyz="0 0 0" rpy="-1.5707 0 -1.5707"/>
+    <parent link="camera"/>
+    <child link="camera_link_optical"/>
+  </joint>
+  <link name="camera_link_optical">
+  </link>
+  <!-- Hokuyo -->
   <link name="hokuyo">
     <pose>0 0 0 0 0 0</pose>
@@ -178,5 +187,5 @@
       </geometry>
     </collision>
-	</link>
+  </link>
   <joint type="fixed" name="hokuyo_joint">
     <origin xyz="0.15 0 0.1" rpy="0 0 0"/>
@@ -187,4 +196,5 @@
     <dynamics damping="1.0" friction="1.0"/>
   </joint>
+  <!-- Colors -->
   <gazebo reference="chassis">
     <material>Gazebo/Grey</material>

Commit message: Add files via upload

File: catkin_ws/src/my_robot/urdf/my_robot.xacro (robot description, xacro)
@@ -157,10 +157,16 @@
   </joint>
   <joint name="camera_optical_joint" type="fixed">
-    <origin xyz="0 0 0" rpy="-1.5707 0 -1.5707"/>
+    <!--<origin xyz="0 0 0" rpy="-1.5707 0 -1.5707"/>-->
+    <origin xyz="0 0 0" rpy="${-pi/2} 0 ${-pi/2}"/>
     <parent link="camera"/>
     <child link="camera_link_optical"/>
   </joint>
-  <link name="camera_link_optical">
-  </link>
+  <link name="camera_link_optical"></link>
+  <!--<link name="camera_rgbd_frame"></link>
+  <joint name="camera_rgbd_joint" type="fixed">
+    <origin xyz="0 0 0" rpy="-${pi/2} 0 -${pi/2}"/>
+    <parent link="camera"/>
+    <child link="camera_rgbd_frame"/>
+  </joint>-->
   <!-- Hokuyo -->
   <link name="hokuyo">
